Commit message: Add: Setup mapping and Nav2, partial hardware setup

File: dash_description/urdf/ros2_control.xacro (robot description, xacro)
@@ -1,17 +1,15 @@
 <?xml version="1.0"?>
 <robot xmlns:xacro="http://www.ros.org/wiki/xacro">
-    <xacro:unless value="$(arg sim_mode)">
-        <ros2_control name="RealRobot" type="system">
+    <ros2_control name="RealRobot" type="system">
             <hardware>
                 <plugin>diffdrive_arduino/DiffDriveArduinoHardware</plugin>
-                <param name="left_wheel_name">left_wheel_joint</param>
-                <param name="right_wheel_name">right_wheel_joint</param>
+                <param name="left_wheel_name">lw_joint</param>
+                <param name="right_wheel_name">rw_joint</param>
                 <param name="loop_rate">30</param>
-                <param name="device">/dev/ttyUSB0</param>
+                <param name="device">/dev/ttyACM0</param>
                 <param name="baud_rate">57600</param>
                 <param name="timeout_ms">1000</param>
-                <param name="enc_counts_per_rev">3436</param>
             </hardware>
-            <joint name="left_wheel_joint">
+            <joint name="lw_joint">
                 <command_interface name="velocity">
                     <param name="min">-10</param>
@@ -21,5 +19,5 @@
                 <state_interface name="velocity"/>
             </joint>
-            <joint name="right_wheel_joint">
+            <joint name="rw_joint">
                 <command_interface name="velocity">
                     <param name="min">-10</param>
@@ -29,34 +27,4 @@
                 <state_interface name="velocity"/>
             </joint>
-        </ros2_control>
-    </xacro:unless>
-    <xacro:if value="$(arg sim_mode)">
-        <ros2_control name="GazeboSystem" type="system">
-            <hardware>
-                <plugin>gz_ros2_control/GazeboSimSystem</plugin>
-            </hardware>
-            <joint name="lw_joint">
-                <command_interface name="velocity">
-                    <param name="min">-10</param>
-                    <param name="max">10</param>
-                </command_interface>
-                <state_interface name="velocity"/>
-                <state_interface name="position"/>
-            </joint>
-            <joint name="rw_joint">
-                <command_interface name="velocity">
-                    <param name="min">-10</param>
-                    <param name="max">10</param>
-                </command_interface>
-                <state_interface name="velocity"/>
-                <state_interface name="position"/>
-            </joint>
-        </ros2_control>
-    </xacro:if>
-    <gazebo>
-        <plugin name="gz_ros2_control::GazeboSimROS2ControlPlugin" filename="libgz_ros2_control-system.so">
-            <parameters>$(find dash_description)/config/my_controllers.yaml</parameters>
-            <parameters>$(find dash_description)/config/gaz_ros2_ctl_use_sim.yaml</parameters>
-        </plugin>
-    </gazebo>
+    </ros2_control>
 </robot>
