Commit message: Update: Working hardware system setup

File: dash_description/urdf/lidar.xacro (robot description, xacro)
@@ -4,9 +4,9 @@
         <parent link="plate3_1"/>
         <child link="laser_frame"/>
-        <origin xyz="-0.055 0.05 0.07" rpy="0 0 3.14"/>
+        <origin xyz="-0.055 0.05 0.07" rpy="0 0 0"/>
     </joint>
     <link name="laser_frame">
         <inertial>
-            <origin xyz="-0.011945780406062 -0.000381929217680526 -0.0170649378129477" rpy="0 0 0" />
+            <origin xyz="-0.011945780406062 -0.000381929217680526 -0.0170649378129477" rpy="0 0 3.14" />
             <mass value="0.073084435549317" />
             <inertia ixx="1.96074931730795E-05" ixy="-3.62091076640009E-07" ixz="4.28230084046735E-07"
@@ -15,5 +15,5 @@
         </inertial>
         <visual>
-            <origin xyz="0 0 0" rpy="0 0 0" />
+            <origin xyz="0 0 0" rpy="0 0 3.14" />
             <geometry>
             <mesh filename="file://$(find dash_description)/meshes/laser_link.STL" />
@@ -22,5 +22,5 @@
         </visual>
         <collision>
-            <origin xyz="0 0 0" rpy="0 0 0" />
+            <origin xyz="0 0 0" rpy="0 0 3.14" />
             <geometry>
             <mesh filename="file://$(find dash_description)/meshes/laser_link.STL" />
